File: FLite40.sch (KiCad schematic (older format))
At the start: 1 part

Commit message: 003_sch01
Parts:
- added C1: 1uF, symbol Device:C_Small
- added C2, C3, C4: 0.1uF, symbol Device:C_Small
- added C5: 10uF, symbol Device:C_Small
- added C6, C7: 22pF, symbol Device:C_Small
- added F1: 500mA, symbol Device:Polyfuse_Small
- added J1: AVR-ISP-6, symbol Connector:AVR-ISP-6
- added R1: 10k, symbol Device:R_Small
- added R2, R3: 22, symbol Device:R_Small
- added R5, R6: 5.1k, symbol Device:R_Small
- added U2: PRTR5V0U2X, symbol random-keyboard-parts:PRTR5V0U2X
- added USB1: HRO-TYPE-C-31-M-12, symbol Type-C:HRO-TYPE-C-31-M-12
- added Y1: 16MHz, symbol Device:Crystal_GND24_Small
- gave numbers to parts that had none: 1
Connections:
- net at U1.10 (PB2): now also J1.4 (MOSI)
- net at U1.11 (PB3): now also J1.1 (MISO)
- net at U1.13 (~RESET): now also J1.5 (~RST)
- net +5V: now reaches U1.14 (VCC), U1.34 (VCC)
- net +5V: now also U1.2 (UVCC), U1.24 (AVCC), U1.44 (AVCC), U1.7 (VBUS), C2.1, C3.1, C4.1, C5.1, F1.1, J1.2 (VCC)
- net GND: now reaches U1.15 (GND), U1.23 (GND), U1.35 (GND), U1.43 (GND)
- net GND: now also U1.5 (UGND), C1.2, C2.2, C3.2, C4.2, C5.2, C6.2, C7.2, J1.6 (GND), R1.1, R5.1, R6.1, U2.1 (GND), USB1.1 (GND), USB1.12 (GND), USB1.13 (SHIELD), Y1.2, Y1.4
- net at U1.16 (XTAL2): now also C7.1, Y1.3
- net at U1.17 (XTAL1): now also C6.1, Y1.1
- net at U1.3 (D-): now also R3.1
- net at U1.33 (~HWB~/PE2): now also R1.2
- net at U1.4 (D+): now also R2.1
- net at U1.6 (UCAP): now also C1.1
- net at U1.9 (PB1): now also J1.3 (SCK)
- new net: R6.2, USB1.10 (CC2)
- new net: R5.2, USB1.4 (CC1)
- new net D+: R2.2, U2.2 (IO1), USB1.6 (DP1), USB1.8 (DP2)
- new net D-: R3.2, U2.3 (IO2), USB1.5 (DN2), USB1.7 (DN1)
- new net VCC: F1.2, U2.4 (VCC), USB1.11 (VBUS), USB1.2 (VBUS)
Other:
- moved on the sheet: U1

Commit message: 004_kairo
Parts:
- removed J1: AVR-ISP-6, symbol Connector:AVR-ISP-6
- added D1, D10, D11, D12, D13, D14, D15, D16, D17, D18, D19, D2, D20, D21, D22, D23, D24, D25, D26, D27, D28, D29, D3, D30, D31, D32, D33, D34, D35, D36, D37, D38, D39, D4, D40, D41, D42, D43, D44, D45, D46, D47, D5, D6, D7, D8, D9: SOD-123, symbol Device:D_Small
- added MX1, MX10, MX11, MX12, MX13, MX14, MX15, MX16, MX17, MX18, MX19, MX2, MX20, MX21, MX22, MX23, MX24, MX25, MX26, MX27, MX28, MX29, MX3, MX30, MX31, MX32, MX33, MX34, MX35, MX36, MX37, MX38, MX39, MX4, MX40, MX41, MX42, MX43, MX44, MX45, MX46, MX47, MX5, MX6, MX7, MX8, MX9: MX-NoLED, symbol MX_Alps_Hybrid:MX-NoLED
- added R4: 10k, symbol Device:R_Small
- added SW1: SW_Push, symbol Switch:SW_Push
Connections:
- net +5V: now also R4.1
- net GND: now also SW1.1
- net at U1.13 (~RESET): now also R4.2, SW1.2
- new net: D2.2 (A), MX2.2 (ROW)
- new net: D1.2 (A), MX1.2 (ROW)
- new net: D3.2 (A), MX3.2 (ROW)
- new net: D4.2 (A), MX4.2 (ROW)
- new net: D5.2 (A), MX5.2 (ROW)
- new net: D6.2 (A), MX6.2 (ROW)
- new net: D7.2 (A), MX7.2 (ROW)
- new net: D8.2 (A), MX8.2 (ROW)
- new net: D9.2 (A), MX9.2 (ROW)
- new net: D10.2 (A), MX10.2 (ROW)
- new net: D11.2 (A), MX11.2 (ROW)
- new net: D12.2 (A), MX12.2 (ROW)
- new net: D13.2 (A), MX13.2 (ROW)
- new net: D25.2 (A), MX25.2 (ROW)
- new net: D24.2 (A), MX24.2 (ROW)
- new net: D23.2 (A), MX23.2 (ROW)
- new net: D22.2 (A), MX22.2 (ROW)
- new net: D21.2 (A), MX21.2 (ROW)
- new net: D20.2 (A), MX20.2 (ROW)
- new net: D19.2 (A), MX19.2 (ROW)
- new net: D18.2 (A), MX18.2 (ROW)
- new net: D17.2 (A), MX17.2 (ROW)
- new net: D16.2 (A), MX16.2 (ROW)
- new net: D14.2 (A), MX14.2 (ROW)
- new net: D15.2 (A), MX15.2 (ROW)
- new net: D36.2 (A), MX36.2 (ROW)
- new net: D35.2 (A), MX35.2 (ROW)
- new net: D34.2 (A), MX34.2 (ROW)
- new net: D33.2 (A), MX33.2 (ROW)
- new net: D32.2 (A), MX32.2 (ROW)
- new net: D31.2 (A), MX31.2 (ROW)
- new net: D30.2 (A), MX30.2 (ROW)
- new net: D29.2 (A), MX29.2 (ROW)
- new net: D28.2 (A), MX28.2 (ROW)
- new net: D27.2 (A), MX27.2 (ROW)
- new net: D37.2 (A), MX37.2 (ROW)
- new net: D26.2 (A), MX26.2 (ROW)
- new net: D47.2 (A), MX47.2 (ROW)
- new net: D46.2 (A), MX46.2 (ROW)
- new net: D45.2 (A), MX45.2 (ROW)
- new net: D44.2 (A), MX44.2 (ROW)
- new net: D43.2 (A), MX43.2 (ROW)
- new net: D42.2 (A), MX42.2 (ROW)
- new net: D41.2 (A), MX41.2 (ROW)
- new net: D40.2 (A), MX40.2 (ROW)
- new net: D38.2 (A), MX38.2 (ROW)
- new net: D39.2 (A), MX39.2 (ROW)
- new net COL0: MX1.1 (COL), MX14.1 (COL), MX38.1 (COL)
- new net COL1: MX15.1 (COL), MX2.1 (COL), MX26.1 (COL), MX39.1 (COL)
- new net COL10: MX11.1 (COL), MX24.1 (COL), MX35.1 (COL), MX45.1 (COL)
- new net COL11: MX12.1 (COL), MX25.1 (COL), MX36.1 (COL), MX46.1 (COL)
- new net COL12: MX13.1 (COL), MX37.1 (COL), MX47.1 (COL)
- new net COL2: MX16.1 (COL), MX27.1 (COL), MX3.1 (COL), MX40.1 (COL)
- new net COL3: MX17.1 (COL), MX28.1 (COL), MX4.1 (COL), MX41.1 (COL)
- new net COL4: MX18.1 (COL), MX29.1 (COL), MX42.1 (COL), MX5.1 (COL)
- new net COL5: MX19.1 (COL), MX30.1 (COL), MX6.1 (COL)
- new net COL6: MX20.1 (COL), MX31.1 (COL), MX43.1 (COL), MX7.1 (COL)
- new net COL7: MX21.1 (COL), MX32.1 (COL), MX8.1 (COL)
- new net COL8: MX22.1 (COL), MX33.1 (COL), MX44.1 (COL), MX9.1 (COL)
- new net COL9: MX10.1 (COL), MX23.1 (COL), MX34.1 (COL)
- new net ROW0: D1.1 (K), D10.1 (K), D11.1 (K), D12.1 (K), D13.1 (K), D2.1 (K), D3.1 (K), D4.1 (K), D5.1 (K), D6.1 (K), D7.1 (K), D8.1 (K), D9.1 (K)
- new net ROW1: D14.1 (K), D15.1 (K), D16.1 (K), D17.1 (K), D18.1 (K), D19.1 (K), D20.1 (K), D21.1 (K), D22.1 (K), D23.1 (K), D24.1 (K), D25.1 (K)
- new net ROW2: D26.1 (K), D27.1 (K), D28.1 (K), D29.1 (K), D30.1 (K), D31.1 (K), D32.1 (K), D33.1 (K), D34.1 (K), D35.1 (K), D36.1 (K), D37.1 (K)
- new net ROW3: D38.1 (K), D39.1 (K), D40.1 (K), D41.1 (K), D42.1 (K), D43.1 (K), D44.1 (K), D45.1 (K), D46.1 (K), D47.1 (K)
Other:
- moved on the sheet: C1, C2, C3, C4, C5, C6, C7, R1, R2, R3, U1, Y1

Commit message: 005_totyu
Parts:
- added J1: AVR-ISP-6, symbol Connector:AVR-ISP-6
Connections:
- net +5V: now also J1.2 (VCC)
- net GND: now also J1.6 (GND)
- net at U1.10 (PB2): now also J1.3 (SCK)
- net RESET: now reaches R4.2, SW1.2, U1.13 (~RESET)
- net RESET: now also J1.5 (~RST)
- net at U1.8 (PB0): now also J1.1 (MISO)
- net at U1.9 (PB1): now also J1.4 (MOSI)
Other:
- note added: "1.25U"
- note added: "1.75U"
- note added: "2.75U"
Changed lines of the file:
@@
 	1    0    0    -1
 $EndComp
+$Comp
+L Connector:AVR-ISP-6 J1
+U 1 1 60637A12
+P 3400 1350
+F 0 "J1" H 3121 1446 50  0000 R CNN
+F 1 "AVR-ISP-6" H 3121 1355 50  0000 R CNN
+F 2 "" V 3150 1400 50  0001 C CNN
+F 3 " ~" H 2125 800 50  0001 C CNN
+	1    3400 1350
+	-1   0    0    -1
+$EndComp
+$Comp
+L power:+5V #PWR0117
+U 1 1 606382CF
+P 3500 850
+F 0 "#PWR0117" H 3500 700 50  0001 C CNN
+F 1 "+5V" H 3515 1023 50  0000 C CNN
+F 2 "" H 3500 850 50  0001 C CNN
+F 3 "" H 3500 850 50  0001 C CNN
+	1    3500 850
+	-1   0    0    -1
+$EndComp
+$Comp
+L power:GND #PWR0118
+U 1 1 606387FC
+P 3500 1750
+F 0 "#PWR0118" H 3500 1500 50  0001 C CNN
+F 1 "GND" H 3505 1577 50  0000 C CNN
+F 2 "" H 3500 1750 50  0001 C CNN
+F 3 "" H 3500 1750 50  0001 C CNN
+	1    3500 1750
+	-1   0    0    -1
+$EndComp
+Text GLabel 1150 1050 2    50   Input ~ 0
+RESET
+Text GLabel 3000 1450 0    50   Input ~ 0
+RESET
+Wire Wire Line
+	2600 1200 2600 1150
+Wire Wire Line
+	2600 1150 3000 1150
+Wire Wire Line
+	2600 1300 2600 1250
+Wire Wire Line
+	2600 1250 3000 1250
+Wire Wire Line
+	2600 1400 2600 1350
+Wire Wire Line
+	2600 1350 3000 1350
+Text Notes 7250 4850 0    50   ~ 0
+2.75U
+Text Notes 8350 4850 0    50   ~ 0
+1.25U
+Text Notes 6150 4850 0    50   ~ 0
+1.25U
+Text Notes 3950 4850 0    50   ~ 0
+1.25U
+Text Notes 4500 4200 0    50   ~ 0
+1.75U
+Text Notes 10550 4200 0    50   ~ 0
+1.25U
+Text Notes 10000 3550 0    50   ~ 0
+1.75U
+Text Notes 3950 3550 0    50   ~ 0
+1.25U
 $EndSCHEMATC

Commit message: 006_kari
Parts:
- added LED1: SK6812MINI, LED_YS-SK6812MINI-E:LED_YS-SK6812MINI-E_ReverseMount_HandSoldering, symbol LED:SK6812MINI
- C1, C2, C3, C4, C5, C6, C7: footprint (none) -> Capacitor_SMD:C_0805_2012Metric_Pad1.15x1.40mm_HandSolder
- D1, D10, D11, D12, D13, D14, D15, D16, D17, D18, D19, D2, D20, D21, D22, D23, D24, D25, D26, D27, D28, D29, D3, D30, D31, D32, D33, D34, D35, D36, D37, D38, D39, D4, D40, D41, D42, D43, D44, D45, D46, D47, D5, D6, D7, D8, D9: footprint (none) -> Diode_SMD:D_SOD-123
- F1: footprint (none) -> Fuse:Fuse_1206_3216Metric
- J1: footprint (none) -> random-keyboard-parts:Reset_Pretty
- MX1, MX10, MX11, MX12, MX13, MX14, MX15, MX16, MX17, MX18, MX19, MX2, MX20, MX21, MX22, MX23, MX24, MX25, MX26, MX27, MX28, MX29, MX3, MX30, MX31, MX32, MX33, MX34, MX35, MX36, MX37, MX38, MX39, MX4, MX40, MX41, MX42, MX43, MX44, MX45, MX46, MX47, MX5, MX6, MX7, MX8, MX9: footprint (none) -> MX_Alps_Hybrid:MX-1U-NoLED
- R1, R2, R3, R4, R5, R6: footprint (none) -> Resistor_SMD:R_0805_2012Metric
- SW1: footprint (none) -> random-keyboard-parts:SKQG-1155865
- U2: footprint (none) -> random-keyboard-parts:SOT143B
- USB1: footprint (none) -> Type-C:HRO-TYPE-C-31-M-12-Assembly
- Y1: footprint (none) -> Crystal:Crystal_SMD_3225-4Pin_3.2x2.5mm
Connections:
- net COL0: now also MX26.1 (COL)
- net COL1: no longer MX26.1 (COL)
- net COL11: no longer MX25.1 (COL)
- net COL12: now also MX25.1 (COL)
- net COL6: no longer MX43.1 (COL)
- net COL7: now also MX43.1 (COL)
- net COL8: no longer MX44.1 (COL)
- net COL9: now also MX44.1 (COL)
- net GND: now also LED1.2 (VSS)
- net VCC: now also LED1.4 (VDD)
- new net LED: LED1.3 (DIN)
- no-connect marks 0 -> 4
Other:
- moved on the sheet: D1, D10, D11, D12, D13, D14, D15, D16, D17, D18, D19, D2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
